Commit message: changed

File: denso_robot_descriptions/vs060_description/vs060.urdf (robot description, URDF)
Before this commit: robot vs060, 8 links, 7 joints
Links:
- added link bucket_link, mass 1; collision mesh filename=package://denso_robot_descriptions/vs060_description/bucket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 scale=1 1 1; visual mesh filename=package://denso_robot_descriptions/vs060_description/bucket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 scale=1 1 1
- added link jig_link, mass 1; collision mesh filename=package://denso_robot_descriptions/vs060_description/jig.stl scale=1 1 1; visual mesh filename=package://denso_robot_descriptions/vs060_description/jig.stl scale=1 1 1
- added link loadcell_link, mass 1; collision mesh filename=package://denso_robot_descriptions/vs060_description/loadce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 scale=1 1 1; visual mesh filename=package://denso_robot_descriptions/vs060_description/loadce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 scale=1 1 1
Joints:
- added joint joint_bucket: type fixed, parent loadcell_link, child bucket_link, origin xyz=0.000000 0.000000 0.000000 rpy=0.000000 0.000000 1.5707963267948966
- added joint joint_jig: type fixed, parent J6, child jig_link, origin xyz=0.000000 0.000000 0.000000 rpy=0.000000 0.000000 0.000000
- added joint joint_loadcell: type fixed, parent jig_link, child loadcell_link, origin xyz=0.000000 0.000000 0.03570 rpy=0.000000 0.000000 0.000000

Commit message: set limit to joint_1 and joint_6

File: denso_robot_descriptions/vs060_description/vs060.urdf (robot description, URDF)
Before this commit: robot vs060, 11 links, 10 joints
Joints:
- joint joint_1: limit lower=-2.96706 upper=2.96706 effort=1 velocity=3.92699081698724 -> lower=-0 upper=0 effort=1 velocity=3.92699081698724
- joint joint_6: limit lower=-6.283185 upper=6.283185 effort=1 velocity=6.28318530717959 -> lower=-0 upper=0 effort=1 velocity=6.28318530717959

Commit message: add joint_4 limit

File: denso_robot_descriptions/vs060_description/vs060.urdf (robot description, URDF)
Before this commit: robot vs060, 11 links, 10 joints
Joints:
- joint joint_4: limit lower=-4.712389 upper=4.712389 effort=1 velocity=3.92699081698724 -> lower=0 upper=0 effort=1 velocity=3.92699081698724

Commit message: fixed get robot state error

File: denso_robot_descriptions/vs060_description/vs060.urdf (robot description, URDF)
Before this commit: robot vs060, 11 links, 10 joints
Joints:
- joint joint_1: limit lower=-0 upper=0 effort=1 velocity=3.92699081698724 -> lower=-0.05 upper=0.05 effort=1 velocity=3.92699081698724
- joint joint_4: limit lower=0 upper=0 effort=1 velocity=3.92699081698724 -> lower=-0.05 upper=0.05 effort=1 velocity=3.92699081698724
- joint joint_6: limit lower=-0 upper=0 effort=1 velocity=6.28318530717959 -> lower=-0.05 upper=0.05 effort=1 velocity=6.28318530717959
